File: 16bit-cpu.kicad_sch (KiCad schematic)
At the start: 0 parts

Commit message: cpu in progress done until out15_c
Parts:
- added R1, R10, R11, R12, R13, R14, R15, R16, R17, R18, R19, R2, R20, R21, R22, R23, R24, R25, R26, R27, R28, R29, R3, R30, R31, R32, R4, R5, R6, R7, R8, R9: 200k, symbol Device:R
- added SW1, SW10, SW11, SW12, SW13, SW14, SW15, SW16, SW17, SW18, SW19, SW2, SW20, SW21, SW22, SW23, SW24, SW25, SW26, SW27, SW28, SW29, SW3, SW30, SW31, SW32, SW4, SW5, SW6, SW7, SW8, SW9: SW_SPST, symbol Switch:SW_SPST
- added U1, U2: ~, symbol symbols:TC74HC00A
Connections:
- new net +5V: SW1.1 (A), SW10.1 (A), SW11.1 (A), SW12.1 (A), SW13.1 (A), SW14.1 (A), SW15.1 (A), SW16.1 (A), SW17.1 (A), SW18.1 (A), SW19.1 (A), SW2.1 (A), SW20.1 (A), SW21.1 (A), SW22.1 (A), SW23.1 (A), SW24.1 (A), SW25.1 (A), SW26.1 (A), SW27.1 (A), SW28.1 (A), SW29.1 (A), SW3.1 (A), SW30.1 (A), SW31.1 (A), SW32.1 (A), SW4.1 (A), SW5.1 (A), SW6.1 (A), SW7.1 (A), SW8.1 (A), SW9.1 (A), U1.14 (Vcc), U2.14 (Vcc)
- new net GND: R1.2, R10.2, R11.2, R12.2, R13.2, R14.2, R15.2, R16.2, R17.2, R18.2, R19.2, R2.2, R20.2, R21.2, R22.2, R23.2, R24.2, R25.2, R26.2, R27.2, R28.2, R29.2, R3.2, R30.2, R31.2, R32.2, R4.2, R5.2, R6.2, R7.2, R8.2, R9.2, U1.7 (GND), U2.7 (GND)
- new net O15_C: U2.11 (4Y)
- new net O15_C_1: U2.12 (4A), U2.13 (4B), U2.6 (2Y)
- new net O16: U2.3 (1Y)
- new net O16_1: U1.11 (4Y), U2.1 (1A)
- new net O16_2: U1.8 (3Y), U2.2 (1B)
- new net SW1: R1.1, SW1.2 (B)
- new net SW10: R10.1, SW10.2 (B)
- new net SW11: R11.1, SW11.2 (B)
- new net SW12: R12.1, SW12.2 (B)
- new net SW13: R13.1, SW13.2 (B)
- new net SW14: R14.1, SW14.2 (B)
- new net SW15: R15.1, SW15.2 (B)
- new net SW16: R16.1, SW16.2 (B), U1.1 (1A), U1.13 (4B), U1.2 (1B), U2.4 (2A)
- new net SW16_NOT: U1.10 (3B), U1.3 (1Y)
- new net SW17: R17.1, SW17.2 (B)
- new net SW18: R18.1, SW18.2 (B)
- new net SW19: R19.1, SW19.2 (B)
- new net SW2: R2.1, SW2.2 (B)
- new net SW20: R20.1, SW20.2 (B)
- new net SW21: R21.1, SW21.2 (B)
- new net SW22: R22.1, SW22.2 (B)
- new net SW23: R23.1, SW23.2 (B)
- new net SW24: R24.1, SW24.2 (B)
- new net SW25: R25.1, SW25.2 (B)
- new net SW26: R26.1, SW26.2 (B)
- new net SW27: R27.1, SW27.2 (B)
- new net SW28: R28.1, SW28.2 (B)
- new net SW29: R29.1, SW29.2 (B)
- new net SW3: R3.1, SW3.2 (B)
- new net SW30: R30.1, SW30.2 (B)
- new net SW31: R31.1, SW31.2 (B)
- new net SW32: R32.1, SW32.2 (B), U1.4 (2A), U1.5 (2B), U1.9 (3A), U2.5 (2B)
- new net SW32_NOT: U1.12 (4A), U1.6 (2Y)
- new net SW4: R4.1, SW4.2 (B)
- new net SW5: R5.1, SW5.2 (B)
- new net SW6: R6.1, SW6.2 (B)
- new net SW7: R7.1, SW7.2 (B)
- new net SW8: R8.1, SW8.2 (B)
- new net SW9: R9.1, SW9.2 (B)
- no-connect marks 0 -> 3

Commit message: finished until SW31_O15_C_AND
Parts:
- added U3, U4, U5, U6, U7, U8, U9: ~, symbol symbols:TC74HC00A
Connections:
- net O15_C: now also U4.12 (4A), U5.12 (4A)
- net SW15: now also U2.10 (3B), U2.9 (3A), U3.4 (2A), U5.1 (1A)
- net SW31: now also U3.1 (1A), U3.12 (4A), U3.2 (1B), U5.13 (4B), U5.2 (1B)
- net SW15_NOT: now reaches U2.8 (3Y)
- net SW15_NOT: now also U3.13 (4B)
- net O15_C_1 renamed O15_C_NOT
- net O15_C_NOT: now also U4.5 (2B)
- new net: U5.10 (3B), U5.11 (4Y), U5.9 (3A)
- new net: U5.3 (1Y), U5.4 (2A), U5.5 (2B)
- new net O15: U4.8 (3Y)
- new net O15_1: U3.10 (3B), U3.6 (2Y)
- new net O15_2: U3.11 (4Y), U3.9 (3A)
- new net O15_3: U3.8 (3Y), U4.1 (1A), U4.2 (1B), U4.4 (2A)
- new net O15_3_NOT: U4.13 (4B), U4.3 (1Y)
- new net O15_4: U4.10 (3B), U4.6 (2Y)
- new net O15_5: U4.11 (4Y), U4.9 (3A)
- new net SW15_SW31_AND: U5.6 (2Y)
- new net SW31_NOT: U3.3 (1Y), U3.5 (2B)
- new net SW31_O15_C_AND: U5.8 (3Y)
- no-connect marks 3 -> 0
